Commit message: Fixed arm lidar, changed Wrench to WrenchStamped, modified front bumper collision, modified wheel friction parameters, changed camera color, added teleop package for easier push to Technion.

File: tec_description/urdf/components/firefly.urdf.xacro (robot description, xacro)
@@ -38,8 +38,7 @@
 				<origin xyz="0 0 0" rpy="0 0 0" />
 				<geometry>
-                    <!-- The mesh is included with the sensor mast mesh -->
 					<box size="0.02 0.02 0.02" />
 				</geometry>
-				<material name="White" />
+				<material name="Black" />
 			</visual>
             <visual>
@@ -48,5 +47,5 @@
 					<cylinder radius="0.0025" length="0.0025" />
 				</geometry>
-				<material name="White" />
+				<material name="Black" />
 			</visual>
 			<collision>
@@ -56,5 +55,5 @@
 					<box size="0.02 0.02 0.02" />
 				</geometry>
-				<material name="White" />
+				<material name="Black" />
 			</collision>
             <collision>
@@ -63,9 +62,9 @@
 					<cylinder radius="0.0025" length="0.0025" />
 				</geometry>
-				<material name="White" />
+				<material name="Black" />
 			</collision>
         </link>
         <gazebo reference="${name}_camera_base_link">
-            <material>Gazebo/WhiteGlow</material>
+            <material>Gazebo/FlatBlack</material>
         </gazebo>
         <gazebo reference="${name}_camera_base_link">

File: tec_description/urdf/lwa_husky.urdf.xacro (robot description, xacro)
@@ -28,5 +28,4 @@
     <xacro:include filename="$(find tec_description)/urdf/utils/parts.urdf.xacro" />
     <!-- sensors -->
-    <xacro:include filename="$(find pr2_description)/urdf/sensors/microstrain_3dmgx2_imu.urdf.xacro" />
     <xacro:include filename="$(find tec_description)/urdf/components/kinect.urdf.xacro" />
     <xacro:include filename="$(find tec_description)/urdf/components/lms151.urdf.xacro" />
@@ -71,5 +70,5 @@
     </gazebo>
     <joint name="base_footprint_joint" type="fixed">
-		<origin xyz="0 0 ${wheel_x_size/2 - base_z_origin_to_wheel_origin}" rpy="0 0 0" />
+        <origin xyz="0 0 ${wheel_x_size/2 - base_z_origin_to_wheel_origin}" rpy="0 0 0" />
         <parent link="base_footprint"/>
         <child link="base_link" />
@@ -128,7 +127,7 @@
         </gazebo>
         <!-- Bumpers -->
-        <tec_part parent="base_footprint" name="front_bumper" visual="bumper" collision="bumper"
+        <tec_part parent="base_footprint" name="front_bumper" visual="front_bumper" collision="front_bumper"
               colour="DarkGray"
-              translateX="0.480" translateY="0.0" translateZ="${0.091 + wheel_x_size/2 - base_z_origin_to_wheel_origin}"
+              translateX="0.530" translateY="0.0" translateZ="${0.091 + wheel_x_size/2 - base_z_origin_to_wheel_origin}"
               rotateX="0.0" rotateY="0.0" rotateZ="0.0"/>
         <gazebo reference="base_footprint_front_bumper_part">
@@ -173,5 +172,5 @@
         <tec_part parent="base_footprint_front_bumper_part" name="sick_bracket" visual="lidar_mount" collision="lidar_mount"
             colour="DarkGray"
-            translateX="-0.075" translateY="0" translateZ="0"
+            translateX="-0.12" translateY="0" translateZ="0"
             rotateX="0" rotateY="0.0" rotateZ="0"/>
         <gazebo reference="flir_ptu_mount_link_sick_bracket_part">
@@ -187,26 +186,45 @@
         </xacro:sensor_firefly>
         <!-- IMU -->
-	<gazebo>
-	  <plugin name="imu_controller" filename="libgazebo_ros_imu.so">
-		<alwaysOn>true</alwaysOn>
-		<updateRate>50.0</updateRate>
-		<bodyName>base_link</bodyName>
-		<topicName>imu/data</topicName>
-		<gaussianNoise>2.89e-08</gaussianNoise>
-	  </plugin>
-	</gazebo>
+        <link name="imu_link">
+           <inertial>
+                <mass value="1e-5" />
+                <origin xyz="0 0 0" rpy="0 0 0"/>
+                <inertia ixx="1e-6" ixy="0" ixz="0" iyy="1e-6" iyz="0" izz="1e-6" />
+            </inertial>
+        </link>
+        <joint name="imu_joint" type="fixed">
+            <origin xyz="0 0 0" rpy="${M_PI/2} ${M_PI/2} 0" />
+            <parent link="base_link"/>
+            <child link="imu_link" />
+        </joint>
+        <gazebo>
+		  <plugin name="imu_controller" filename="libhector_gazebo_ros_imu.so">
+			<alwaysOn>true</alwaysOn>
+			<updateRate>50.0</updateRate>
+			<bodyName>imu_link</bodyName>
+			<topicName>imu/data</topicName>
+            <accelDrift>0.005 0.005 0.005</accelDrift>
+            <accelGaussianNoise>0.005 0.005 0.005</accelGaussianNoise>
+            <rateDrift>0.005 0.005 0.005 </rateDrift>
+            <rateGaussianNoise>0.005 0.005 0.005 </rateGaussianNoise>
+            <headingDrift>0.005</headingDrift>
+            <headingGaussianNoise>0.005</headingGaussianNoise>
+		  </plugin>
+		</gazebo>
         <!-- GPS -->
         <gazebo>
-            <plugin name="gps_controller" filename="libgazebo_ros_p3d.so">
-            <alwaysOn>true</alwaysOn>
-            <updateRate>30.0</updateRate>
-            <bodyName>base_link</bodyName>
-            <topicName>gps/fix</topicName>
-            <gaussianNoise>0.05</gaussianNoise>
+            <plugin name="gps_controller" filename="libhector_gazebo_ros_gps.so">
+                <updateRate>1</updateRate>
+                <robotNamespace>gps</robotNamespace>
+                <bodyName>base_link</bodyName>
+                <velocityTopicName>vo</velocityTopicName>
+                <referenceLatitude>32.7</referenceLatitude>
+                <referenceLongitude>35.02</referenceLongitude>
+                <drift>0.0001 0.0001 0.0001</drift>
             </plugin>
         </gazebo>
         <!-- Arm Lidar -->
         <xacro:sensor_hokuyo parent="arm_gripper" name="hokuyo">
-            <origin xyz="-0.06 0 0.105" rpy="0 0 0"/>
+            <origin xyz="-0.06 0 0.105" rpy="0 -0.001 0"/>
         </xacro:sensor_hokuyo>
         <!-- Arm Camera -->

File: tec_description/urdf/utils/wheel.urdf.xacro (robot description, xacro)
@@ -76,9 +76,9 @@
 		</link>
 		<gazebo reference="${fb}_${lr}_wheel">
-			<mu1 value="1.0"/>
-			<mu2 value="1.0"/>
+            <fdir1 value="1 0 0"/>
+			<mu1 value="250.0"/>
+            <mu2 value="0.1"/>
 			<kp  value="10000000.0" />
 			<kd  value="1.0" />
-			<fdir1 value="1 0 0"/>
 			<material>Gazebo/Grey</material>
 			<turnGravityOff>false</turnGravityOff>
